Commit message: sdf model

File: urdf/t265_car.urdf.xacro (robot description, xacro)
@@ -9,5 +9,5 @@
     </joint>  -->
   <xacro:realsense_T265 sensor_name="camera" parent_link="base_link" rate="10.0">
-    <origin rpy="1.57 1.57 0" xyz="0.155 0 0.05"/>
+    <origin rpy="1.57 1.57 0" xyz="0.235 0 0.055"/>
   </xacro:realsense_T265>
     <gazebo>
